File: board-files-eagle/mavroOBD/mavroOBD.sch (EAGLE design)
At the start: 27 parts, among them Q1 8mhz / 490-1198-1-ND, Q2 16mhz / 490-1198-1-ND, U1 ATMEGA328, U3 MCP2551, U4 MCP2515

Commit message: Fixed Tag Connect ISP pin assignments
Connections:
- net CS: no longer J1.ICSP_DAT/PGD
- net D9: no longer J1.VSS(GND)
- net MISO: now also J1.VPP/MCLR
- net MOSI: now also J1.ICSP_DAT/PGD; no longer J1.VPP/MCLR
- net SCK: now also J1.VSS(GND)
Changed lines of the file:
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@@
 <label x="73.66" y="74.93" size="1.27" layer="95" xref="yes"/>
+</segment>
+<segment>
+<pinref part="J1" gate="G$1" pin="VSS(GND)"/>
+<wire x1="220.98" y1="175.26" x2="210.439" y2="175.26" width="0.1524" layer="91"/>
+<label x="210.566" y="175.26" size="1.27" layer="95" rot="R180" xref="yes"/>
 </segment>
 </net>
@@
 <label x="73.66" y="80.01" size="1.27" layer="95" xref="yes"/>
 </segment>
+<segment>
+<pinref part="J1" gate="G$1" pin="VPP/MCLR"/>
+<wire x1="220.98" y1="180.34" x2="210.82" y2="180.34" width="0.1524" layer="91"/>
+<label x="210.82" y="180.34" size="1.27" layer="95" rot="R180" xref="yes"/>
+</segment>
 </net>
 <net name="MOSI" class="0">
@@
 </segment>
 <segment>
-<pinref part="J1" gate="G$1" pin="VPP/MCLR"/>
-<wire x1="220.98" y1="180.34" x2="210.82" y2="180.34" width="0.1524" layer="91"/>
-<label x="210.82" y="180.34" size="1.27" layer="95" rot="R180" xref="yes"/>
+<pinref part="J1" gate="G$1" pin="ICSP_DAT/PGD"/>
+<wire x1="220.98" y1="172.72" x2="210.82" y2="172.72" width="0.1524" layer="91"/>
+<label x="210.82" y="172.72" size="1.27" layer="95" rot="R180" xref="yes"/>
 </segment>
 </net>
@@
 <label x="198.12" y="88.9" size="1.27" layer="95" rot="R180" xref="yes"/>
 </segment>
-<segment>
-<pinref part="J1" gate="G$1" pin="VSS(GND)"/>
-<wire x1="220.98" y1="175.26" x2="210.439" y2="175.26" width="0.1524" layer="91"/>
-<label x="210.566" y="175.26" size="1.27" layer="95" rot="R180" xref="yes"/>
-</segment>
 </net>
 <net name="D8" class="0">
@@
 <label x="223.52" y="106.68" size="1.27" layer="95" xref="yes"/>
 </segment>
-<segment>
-<pinref part="J1" gate="G$1" pin="ICSP_DAT/PGD"/>
-<wire x1="220.98" y1="172.72" x2="210.82" y2="172.72" width="0.1524" layer="91"/>
-<label x="210.82" y="172.72" size="1.27" layer="95" rot="R180" xref="yes"/>
-</segment>
-</net>
+</net>

Commit message: REV 3 Board - Sent to OSHPark
Fixed a few via sizes, added VCC to ISP pin and REV 3 to silkscreen.
Parts:
- Q1: value 8mhz / 490-1198-1-ND -> 16mhz / 490-1198-1-ND
Connections:
- removed net 3.3V: J1.VDD
- net VCC: now also J1.VDD
Changed lines of the file:
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@@
 <part name="C2" library="SparkFun" deviceset="CAP" device="0603-CAP" value="0.1uF"/>
 <part name="U$3" library="SparkFun" deviceset="OSHW-LOGO" device="S"/>
-<part name="Q1" library="Testing" deviceset="RESONATOR" device="1:1" value="8mhz / 490-1198-1-ND"/>
+<part name="Q1" library="Testing" deviceset="RESONATOR" device="1:1" value="16mhz / 490-1198-1-ND"/>
 <part name="U3" library="IC" deviceset="MCP2551" device="-SOIC8" value="MCP2551"/>
 <part name="U4" library="IC" deviceset="MCP2515" device="-SOIC18" value="MCP2515"/>
@@
 <pinref part="VCC1" gate="G$1" pin="3.3V"/>
 </segment>
+<segment>
+<pinref part="J1" gate="G$1" pin="VDD"/>
+<wire x1="220.98" y1="177.8" x2="205.74" y2="177.8" width="0.1524" layer="91"/>
+<label x="213.36" y="177.8" size="1.778" layer="95"/>
+<pinref part="P+6" gate="G$1" pin="3.3V"/>
+</segment>
 </net>
 <net name="D9" class="0">
@@
 </segment>
 </net>
-<net name="3.3V" class="1">
-<segment>
-<pinref part="J1" gate="G$1" pin="VDD"/>
-<wire x1="220.98" y1="177.8" x2="205.74" y2="177.8" width="0.1524" layer="91"/>
-<label x="213.36" y="177.8" size="1.778" layer="95"/>
-<pinref part="P+6" gate="G$1" pin="3.3V"/>
-</segment>
-</net>
